Commit message: added (small) urdf files to world

File: src/asl_turtlebot/models/box_carrot/box_carrot.urdf (robot description, URDF)
Before this commit: robot ar_2020, 1 links, 0 joints
Links:
- link simple_box_base_link: geometry collision box size=0.2 0.2 0.2; visual mesh filename=package://asl_turtlebot/models/box_carrot/box_carrot.dae

File: src/asl_turtlebot/models/box_fence/box_fence.urdf (robot description, URDF)
Before this commit: robot ar_2020, 1 links, 0 joints
Links:
- link simple_box_base_link: geometry collision box size=0.2 0.2 0.2; visual mesh filename=package://asl_turtlebot/models/box_fence/box_fence.dae

File: src/asl_turtlebot/models/box_house/box_house.urdf (robot description, URDF)
Before this commit: robot ar_2020, 1 links, 0 joints
Links:
- link simple_box_base_link: geometry collision box size=0.2 0.2 0.2; visual mesh filename=package://asl_turtlebot/models/box_house/box_house.dae

File: src/asl_turtlebot/models/box_mountain/box_mountain.urdf (robot description, URDF)
Before this commit: robot ar_2020, 1 links, 0 joints
Links:
- link simple_box_base_link: geometry collision box size=0.2 0.2 0.2; visual mesh filename=package://asl_turtlebot/models/box_mountain/box_mountain.dae

File: src/asl_turtlebot/models/box_toilet/box_toilet.urdf (robot description, URDF)
Before this commit: robot ar_2020, 1 links, 0 joints
Links:
- link simple_box_base_link: geometry collision box size=0.2 0.2 0.2; visual mesh filename=package://asl_turtlebot/models/box_toilet/box_toilet.dae
