Commit message: more debugging full pipeline

File: src/asl_turtlebot/models/box_apple/box_apple.urdf (robot description, URDF)
Before this commit: robot ar_2020, 1 links, 0 joints
Links:
- link simple_box_base_link: geometry collision box size=0.25 0.50 0.1; visual mesh filename=package://asl_turtlebot/models/box_apple/box_apple.dae

File: src/asl_turtlebot/models/box_apple1/box_apple1.urdf (robot description, URDF)
Before this commit: robot ar_2020, 1 links, 0 joints
Links:
- link simple_box_base_link: geometry collision box size=0.25 0.50 0.1; visual mesh filename=package://asl_turtlebot/models/box_apple1/box_apple1.dae

File: src/asl_turtlebot/models/box_cake/box_cake.urdf (robot description, URDF)
Before this commit: robot ar_2020, 1 links, 0 joints
Links:
- link simple_box_base_link: geometry collision box size=0.25 0.50 0.1; visual mesh filename=package://asl_turtlebot/models/box_cake/box_cake.dae

File: src/asl_turtlebot/models/box_doughnut/box_doughnut.urdf (robot description, URDF)
Before this commit: robot ar_2020, 1 links, 0 joints
Links:
- link simple_box_base_link: geometry collision box size=0.25 0.50 0.1; visual mesh filename=package://asl_turtlebot/models/box_doughnut/box_doughnut.dae

File: src/asl_turtlebot/models/box_orange/box_orange.urdf (robot description, URDF)
Before this commit: robot ar_2020, 1 links, 0 joints
Links:
- link simple_box_base_link: geometry collision box size=0.25 0.50 0.12; visual mesh filename=package://asl_turtlebot/models/box_orange/box_orange.dae

File: src/asl_turtlebot/models/box_pizza/box_pizza.urdf (robot description, URDF)
Before this commit: robot ar_2020, 1 links, 0 joints
Links:
- link simple_box_base_link: geometry collision box size=0.25 0.50 0.1; visual mesh filename=package://asl_turtlebot/models/box_pizza/box_pizza.dae
